File: saturation_meter.kicad_pcb (KiCad board)
At the start: 2 copper layers, 138 x 111 mm, 64 parts, among them J1 Vin, J2 DUT, J3 Inputs, J4 Outputs, J5 UC, Q1 BUK556, Q2 BUK556, Q3 BC328, U1 LF33_TO220, U2 IR2112

Commit message: Updated to double layer
Parts:
- added ?: , , F.Cu at (163.0, 79.0)
- added ?: , , F.Cu at (204.0, 113.0)
- added ?: , , F.Cu at (159.0, 79.0)
- added ?: , , F.Cu at (148.0, 123.5)
- added ?: , , F.Cu at (155.0, 79.0)
- added ?: , , F.Cu at (208.5, 110.5)
- added ?: , , F.Cu at (167.0, 79.0)
- added ?: , , F.Cu at (105.5, 134.5)
- added ?: , , F.Cu at (213.0, 113.0)
- added ?: , , F.Cu at (171.0, 79.0)
- added R20: 100k, Resistor_THT:R_Axial_DIN0207_L6.3mm_D2.5mm_P10.16mm_Horizontal, F.Cu at (181.0, 81.7)
- moved H5 1.50 mm to (147.5, 81.5)
- moved C1 0.12 mm to (97.5, 61.0)
- moved C10 0.12 mm to (179.0, 132.5)
- moved C11 0.12 mm to (101.5, 111.5)
- moved C2 0.12 mm to (132.5, 61.0)
- moved C3 0.12 mm to (165.5, 61.0)
- moved C4 0.12 mm to (198.5, 61.0)
- moved C5 0.12 mm to (140.0, 133.5)
- moved C6 0.12 mm to (156.0, 133.5)
- moved C7 0.12 mm to (179.0, 125.5)
- moved C8 0.12 mm to (91.5, 108.0)
- moved C9 0.12 mm to (96.0, 112.5)
- moved D1 0.12 mm to (84.5, 99.6)
- moved D2 0.12 mm to (187.5, 75.9)
- moved D3 0.12 mm to (115.0, 78.5)
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Routing:
- net /driver_ho: track 0.00 -> 11.0 mm
- net Net-(Q3-B): track 0.00 -> 6.86 mm
- net Net-(Q3-C): track 0.00 -> 5.82 mm
- added copper zone on F.Cu, net GND

Commit message: Updated to v1.1.0 fixed, shutdown of ir2112, added enclosure
Parts:
- removed the ? at (171.0, 79.0)
- removed Q3: BC328, Package_TO_SOT_THT:TO-92_Inline
- added ?: , , F.Cu at (151.0, 46.5)
- added ?: , , F.Cu at (92.0, 77.0)
- added ?: , , F.Cu at (200.8, 74.5)
- added ?: , , F.Cu at (113.0, 48.2)
- added ?: , , F.Cu at (204.8, 74.5)
- added ?: , , F.Cu at (147.0, 46.5)
- added ?: , , F.Cu at (180.0, 46.5)
- added ?: , , F.Cu at (92.0, 73.0)
- added ?: , , F.Cu at (212.8, 74.5)
- added ?: , , F.Cu at (117.0, 48.2)
- added ?: , , F.Cu at (184.0, 46.5)
- added ?: , , F.Cu at (208.8, 74.5)
- added D7: 1N4007, Diode_THT:D_DO-41_SOD81_P10.16mm_Horizontal, F.Cu at (82.8, 103.8)
- added Q4: BC638, Package_TO_SOT_THT:TO-92_Inline, F.Cu at (95.5, 98.0)
- added REF**: Strap_P5.08mm_Horizontal, strap:Strap_P5.08mm_Horizontal, F.Cu at (115.0, 112.0)
- R20: value 100k -> 8k2
- REF** (x9): value R_Axial_DIN0207_L6.3mm_D2.5mm_P15.24mm_Horizontal -> Strap_P15.24mm_Horizontal; footprint Resistor_THT:R_Axial_DIN0207_L6.3mm_D2.5mm_P15.24mm_Horizontal -> strap:Strap_P15.24mm_Horizontal
- REF** (x2): value R_Axial_DIN0204_L3.6mm_D1.6mm_P5.08mm_Horizontal -> Strap_P5.08mm_Horizontal; footprint Resistor_THT:R_Axial_DIN0204_L3.6mm_D1.6mm_P5.08mm_Horizontal -> strap:Strap_P5.08mm_Horizontal
- moved R19 25.5 mm to (90.0, 124.2), turned to 90 degrees
- moved R14 10.2 mm to (99.1, 92.5), turned to 180 degrees
- moved J2 5.27 mm to (137.8, 94.0)
- moved REF** 4.87 mm to (140.0, 120.8)
- moved REF** 4.66 mm to (156.0, 120.8)
- moved R17 4.25 mm to (108.7, 141.5)
- moved J5 3.50 mm to (86.5, 114.0)
- moved R16 3.04 mm to (95.5, 133.2)
- moved R13 2.96 mm to (98.5, 130.5)
Connections:
- J3 pad 1: /hin_uc -> /sd_uc
- J3 pad 2: /sd_uc -> /hin_uc
- R19 pad 1: GND -> /sd_uc
- R19 pad 2: /sd_uc -> +3.3V
Routing:
- net +3.3V: track 23.8 -> 31.0 mm
- net /vin_prot: track 81.6 -> 87.6 mm
- net /hin_uc: track 12.7 -> 18.5 mm
- net Net-(D6-A): track 11.6 -> 6.78 mm
- net /sd_uc: track 15.9 -> 20.3 mm
- net /sd: track 6.41 -> 9.44 mm
- net /hin: track 9.40 -> 6.44 mm
- net Net-(Q4-C): track 5.82 -> 8.35 mm
- net /driver_ho: track 11.0 -> 13.4 mm
- net /high_nmos_s: track 60.4 -> 58.3 mm
- net /low_nmos_d: track 21.7 -> 23.1 mm
Other:
- board text added: "1.1.0"
- board text removed: "1.0.0"
